Commit message: Fix Gazebo physics glitches, optimize URDF collision, fix model download hang, and add README

File: src/zmr_gazebo/urdf/zmr_robot_sim.urdf (robot description, URDF)
Before this commit: robot zmr_robot, 7 links, 6 joints
Links:
- removed link caster_front
- removed link caster_rear
- added link caster_fl, mass 0.2; collision sphere radius=0.030; visual sphere radius=0.033
- added link caster_fr, mass 0.2; collision sphere radius=0.030; visual sphere radius=0.033
- added link caster_rl, mass 0.2; collision sphere radius=0.030; visual sphere radius=0.033
- added link caster_rr, mass 0.2; collision sphere radius=0.030; visual sphere radius=0.033
- link base_link: mass 10.0 -> 15.0; geometry collision box size=0.95 0.65 0.18; visual box size=0.95 0.65 0.18
Joints:
- removed joint caster_front_joint
- removed joint caster_rear_joint
- added joint caster_fl_joint: type fixed, parent base_link, child caster_fl, origin xyz=0.4575 0.2875 0.0 rpy=0 0 0
- added joint caster_fr_joint: type fixed, parent base_link, child caster_fr, origin xyz=0.4575 -0.2875 0.0 rpy=0 0 0
- added joint caster_rl_joint: type fixed, parent base_link, child caster_rl, origin xyz=-0.4575 0.2875 0.0 rpy=0 0 0
- added joint caster_rr_joint: type fixed, parent base_link, child caster_rr, origin xyz=-0.4575 -0.2875 0.0 rpy=0 0 0
- joint left_wheel_joint: origin xyz=0.0 0.263 0.047 rpy=-1.5707963 0 0 -> xyz=-0.035 0.263 0.047 rpy=-1.5707963 0 0
- joint right_wheel_joint: origin xyz=0.0 -0.263 0.047 rpy=-1.5707963 0 0 -> xyz=-0.035 -0.263 0.047 rpy=-1.5707963 0 0
