Commit message: Version 2.0: Headless 2D Simulator, SLAM Toolbox, Nav2 Autonomous Navigation, RViz Visualization, and URDF Calibration

File: src/zmr_description/urdf/zmr_robot.urdf (robot description, URDF)
Before this commit: robot zmr_robot, 14 links, 13 joints
Joints:
- joint base_footprint_to_base_link: origin xyz=0 0 0 rpy=0 0 0 -> xyz=0 0 0.070 rpy=0 0 0
- joint base_to_right_wheel: axis 0 0 1 -> 0 0 -1
